File: examples/voice-buddy/pcb/kicad/voicebuddy.place.kicad_pcb (KiCad board)
At the start: 2 copper layers, 70 x 70 mm, 66 parts, among them J1 USB-C-16P, J2 SPK-4ohm-3W, J3 OLED-SSD1306-0.96, SW1 BOOT, SW2 VOL-, SW3 VOL+, U1 ESP32-S3-WROOM-1-N16R8, U2 ES8311, U3 ES7210, U4 NS4150B, U5 AMS1117-3.3, U6 USBLC6-2SC6

Commit message: docs + housekeeping: voice-buddy is the worked end-to-end example
Roadmap Phase 1 checked off via voice-buddy; README flagship entry; CHANGELOG
for pcblib / cad scripts / plm cross-checks / the example; AGENTS.md gains the
placement-scorecard gate line and the committed-contract-artifact carve-out;
gitignore covers autoroute work dirs, stage boards and reports; pager-buddy's
two real strapping-pin uses (GPIO45/46) acknowledged with strap_ok so the new
plm lint reads clean. Adds the voice-buddy brief, README, selftest firmware
skeleton and per-dir gitignore.

Co-Authored-By: Claude Fable 5 <noreply@anthropic.com>
Claude-Session: https://claude.ai/code/session_01Y8ubvNoye4BCDfZE93wu9N
Parts:
- moved C19 15.0 mm to (125.5, 145.0)
- moved C20 15.0 mm to (125.5, 148.4)
- moved C11 2.06 mm to (111.8, 133.0), turned to 0 degrees

Commit message: voice-buddy: routing WIP + a hard-won gate lesson; honest status everywhere
drc_report.py's GUI-style report ('Severity: error') never matched
pcb_check.sh's kicad-cli-style '; error' grep — the DRC gate read 444 real
violations as ZERO, and routing proceeded on phantom-clean boards. The
fallback now normalizes its output, design-rules.md records the
run-a-deliberate-short-first rule, and every premature 'DRC 0/0' claim in
README/roadmap/CHANGELOG/product.yaml is corrected to the true state:
placement gates green, scripted routing (power/locals/audio/mics/speaker
chunks in routing.py) in progress, DRC not yet clean. Also: channel-keeping
placement fixes (C11/C12/C13/C17/C26 out of the bus channel), +5V amp riser
moved to F.Cu.

Co-Authored-By: Claude Fable 5 <noreply@anthropic.com>
Claude-Session: https://claude.ai/code/session_01Y8ubvNoye4BCDfZE93wu9N
Parts:
- moved C12 16.7 mm to (123.6, 138.5), turned to 90 degrees
- moved C13 12.2 mm to (121.3, 138.5), turned to 90 degrees
- moved C26 11.8 mm to (117.2, 142.6)
- moved C11 3.98 mm to (115.4, 131.3)
- moved C17 3.13 mm to (114.0, 141.6), turned to 90 degrees
